Commit message: Commit of kuka rsi communication with advanced manipulation

File: SIMTech_ws/src/industrial_robot_ros_packages/simtech_kuka/simtech_kuka_kr500_support/urdf/kr500r2380_macro.xacro (robot description, xacro)
@@ -1,8 +1,17 @@
 <?xml version="1.0"?>
 <robot xmlns:xacro="http://wiki.ros.org/xacro">
+    <xacro:macro name="default_inertial" params="mass">
+        <inertial>
+            <mass value="${mass}" />
+            <inertia ixx="1.0" ixy="0.0" ixz="0.0"
+                iyy="1.0" iyz="0.0"
+                izz="1.0" />
+            </inertial>
+    </xacro:macro>
   <xacro:include filename="$(find kuka_resources)/urdf/common_constants.xacro"/>
   <xacro:include filename="$(find kuka_resources)/urdf/common_materials.xacro"/>
   <xacro:macro name="kuka_kr500r2380" params="prefix">
     <link name="${prefix}base_link">
+    <xacro:default_inertial mass="1"/>
       <visual>
         <origin xyz="0 0 0" rpy="0 0 0"/>
@@ -20,4 +29,5 @@
     </link>
     <link name="${prefix}link_1">
+    <xacro:default_inertial mass="1"/>
       <visual>
         <origin xyz="0 0 0" rpy="0 0 0"/>
@@ -35,4 +45,5 @@
     </link>
     <link name="${prefix}link_2">
+    <xacro:default_inertial mass="1"/>
       <visual>
         <origin xyz="0 0 0" rpy="0 0 0"/>
@@ -50,4 +61,5 @@
     </link>
     <link name="${prefix}link_3">
+    <xacro:default_inertial mass="1"/>
       <visual>
         <origin xyz="0 0 0" rpy="0 0 0"/>
@@ -65,4 +77,5 @@
     </link>
     <link name="${prefix}link_4">
+    <xacro:default_inertial mass="1"/>
       <visual>
         <origin xyz="0 0 0" rpy="0 0 0"/>
@@ -80,4 +93,5 @@
     </link>
     <link name="${prefix}link_5">
+    <xacro:default_inertial mass="1"/>
       <visual>
         <origin xyz="0 0 0" rpy="0 0 0"/>
@@ -95,4 +109,5 @@
     </link>
     <link name="${prefix}link_6">
+    <xacro:default_inertial mass="1"/>
       <visual>
         <origin xyz="0 0 0" rpy="0 0 0"/>

File: SIMTech_ws/src/industrial_robot_ros_packages/simtech_kuka/simtech_kuka_kr90_support/urdf/LAAM_workcell.xacro (robot description, xacro)
@@ -1,4 +1,4 @@
 <?xml version="1.0" ?>
-<robot name="kr90_machining_workcell" xmlns:xacro="http://ros.org/wiki/xacro">
+<robot name="simtech_kuka_workcell" xmlns:xacro="http://ros.org/wiki/xacro">
   <property name="pi" value="3.141592654" />
   <link name="world"/>
@@ -17,6 +17,6 @@
   </xacro:property>
   <!-- Robot -->
-  <xacro:include filename="$(find simtech_kuka_kr90_support)/urdf/kr90r2700.xacro"/>
-  <joint name="kuka_machining_robot" type="fixed">
+  <xacro:include filename="$(find simtech_kuka_workcell)/urdf/kuka_LAAM_robot.xacro"/>
+  <joint name="kuka_robot" type="fixed">
       <parent link="world"/>
       <child link="base_link"/>
@@ -24,11 +24,11 @@
   </joint>
   <!-- Head -->
-  <xacro:include filename="$(find simtech_kuka_kr90_support)/urdf/spindle.xacro"/>
-  <joint name="spindle_head" type="fixed">
-    <parent link="link_6"/>
-    <child link="spindle_head_link"/>
+  <xacro:include filename="$(find simtech_kuka_workcell)/urdf/head.xacro"/>
+  <joint name="laser_head" type="fixed">
+    <parent link="tool0"/>
+    <child link="laser_head_link"/>
     <!-- <origin xyz="0.14633243 -0.083423 0.172" rpy="${radians(0)} ${radians(180)} 0" /> -->
-    <origin xyz="0 0 0" rpy="${radians(0)} 0 0" />
-    <!-- <origin xyz="-0.14633243 0.083423 0.172" rpy="${radians(0)} ${radians(0)} 0" /> -->
+    <origin xyz="-0.14633243 0.083423 0.172" rpy="${radians(0)} ${radians(180)} ${radians(180)}" />
+    <!-- <origin xyz="0.14633243 -0.083423 0.172" rpy="${radians(0)} ${radians(0)} 0" /> -->
     <axis xyz="0 0 1"/>
   </joint>
